File: public/electronic/integrated-circuit/avr-dx/fade/minimal.kicad_sch (KiCad schematic)
At the start: 11 parts, among them P2 USB_C_Plug_USB2.0, U1 CH340C, U3 AVR128DA28x-xSP

Commit message: Save changes at: 1759505071
Connections:
- net at D1.2 (A): now also U3.22 (PA0); no longer U3.28 (PA6)
Other:
- moved on the sheet: D1, R4
Changed lines of the file:
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@@
+	)
+	(no_connect
+		(at 101.6 106.68)
 	)
 	(no_connect
 		(at 101.6 96.52)
 	)
-	(no_connect
-		(at 101.6 91.44)
-	)
 	(wire
 		(pts
@@
 	(wire
 		(pts
-			(xy 83.82 106.68) (xy 86.36 106.68)
+			(xy 83.82 91.44) (xy 86.36 91.44)
 		)
 		(stroke
@@
 	(wire
 		(pts
+			(xy 93.98 91.44) (xy 101.6 91.44)
+		)
+		(stroke
+			(width 0)
+			(type default)
+		)
+	)
+	(wire
+		(pts
 			(xy 123.19 80.01) (xy 121.92 80.01)
 		)
@@
 	(wire
 		(pts
-			(xy 93.98 106.68) (xy 101.6 106.68)
-		)
-		(stroke
-			(width 0)
-			(type default)
-		)
-	)
-	(wire
-		(pts
 			(xy 184.15 83.82) (xy 190.5 83.82)
 		)
@@
 	(wire
 		(pts
-			(xy 73.66 106.68) (xy 76.2 106.68)
+			(xy 73.66 91.44) (xy 76.2 91.44)
 		)
 		(stroke
@@
 	(symbol
 		(lib_id "Device:LED")
-		(at 90.17 106.68 0)
+		(at 90.17 91.44 0)
 		(unit 1)
 		(exclude_from_sim no)
@@
 		(dnp no)
 		(property "Reference" "D1"
-			(at 90.1954 103.5558 0)
+			(at 90.1954 88.3158 0)
 			(effects
 				(font
@@
 		)
 		(property "Value" "TEST LED"
-			(at 90.1446 111.0996 0)
+			(at 90.1446 95.8596 0)
 			(effects
 				(font
@@
 		)
 		(property "Footprint" ""
-			(at 90.17 106.68 0)
+			(at 90.17 91.44 0)
 			(effects
 				(font
@@
 		)
 		(property "Datasheet" "~"
-			(at 90.17 106.68 0)
+			(at 90.17 91.44 0)
 			(effects
 				(font
@@
 		)
 		(property "Description" ""
-			(at 90.17 106.68 0)
+			(at 90.17 91.44 0)
 			(effects
 				(font
@@
 	(symbol
 		(lib_id "Device:R")
-		(at 80.01 106.68 90)
+		(at 80.01 91.44 90)
 		(mirror x)
 		(unit 1)
@@
 		(dnp no)
 		(property "Reference" "R4"
-			(at 80.01 113.03 90)
+			(at 80.01 97.79 90)
 			(effects
 				(font
@@
 		)
 		(property "Value" "1k"
-			(at 80.01 110.49 90)
+			(at 80.01 95.25 90)
 			(effects
 				(font
@@
 		)
 		(property "Footprint" ""
-			(at 80.01 104.902 90)
+			(at 80.01 89.662 90)
 			(effects
 				(font
@@
 		)
 		(property "Datasheet" "~"
-			(at 80.01 106.68 0)
+			(at 80.01 91.44 0)
 			(effects
 				(font
@@
 		)
 		(property "Description" ""
-			(at 80.01 106.68 0)
+			(at 80.01 91.44 0)
 			(effects
 				(font
@@
 	(symbol
 		(lib_id "power:GND")
-		(at 73.66 106.68 270)
+		(at 73.66 91.44 270)
 		(unit 1)
 		(exclude_from_sim no)
@@
 		(fields_autoplaced yes)
 		(property "Reference" "#PWR011"
-			(at 67.31 106.68 0)
+			(at 67.31 91.44 0)
 			(effects
 				(font
@@
 		)
 		(property "Value" "GND"
-			(at 69.85 106.6799 90)
+			(at 69.85 91.4399 90)
 			(effects
 				(font
@@
 		)
 		(property "Footprint" ""
-			(at 73.66 106.68 0)
+			(at 73.66 91.44 0)
 			(effects
 				(font
@@
 		)
 		(property "Datasheet" ""
-			(at 73.66 106.68 0)
+			(at 73.66 91.44 0)
 			(effects
 				(font
@@
 		)
 		(property "Description" ""
-			(at 73.66 106.68 0)
-			(effects
-				(font
+			(at 73.66 91.44 0)
+			(effects
+				(font
