File: public/electronic/integrated-circuit/avr-dx/dac/minimal.kicad_sch (KiCad schematic)
At the start: 12 parts, among them P2 USB_C_Plug_USB2.0, U1 CH340C, U3 AVR128DA28x-xSP

Commit message: Save changes at: 1759601888
Connections:
- net at R4.2: now also U3.12 (PD6); no longer U3.16 (XTAL32K1/PF0)
Other:
- moved on the sheet: C5, LS1, R4
