File: static/electronic/integrated-circuit/avr-dx/dac/minimal.kicad_sch (KiCad schematic)
At the start: 13 parts, among them P2 USB_C_Plug_USB2.0, U1 CH340C, U3 AVR128DA28x-xSP

Commit message: Save changes at: 1759601888
Parts:
- removed D1, D2: TEST LED, symbol Device:LED
- removed R6: 1k, symbol Device:R
- added C5: 100nF, symbol Device:C
- added LS1: Speaker, symbol Device:Speaker
- renumbered C7 to C1, C6 to C2, C8 to C3
Connections:
- net GND: now also C5.2, LS1.2; no longer R4.1
- net at R4.2: now also U3.12 (PD6)
- new net: C5.1, LS1.1, R4.1
- no-connect marks 31 -> 32
Other:
- moved on the sheet: R4
