File: public/electronic/integrated-circuit/lm386/schematic.kicad_sch (KiCad schematic)
At the start: 12 parts, among them U1 LM386

Commit message: Save changes at: 1779452923
Parts:
- added C5: 1uF, symbol Device:C_Small
Connections:
- net Input: now also C5.1; no longer RV1.1
- new net: C5.2, RV1.1
Changed lines of the file:
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@@
+	(wire
+		(pts
+			(xy 107.95 82.55) (xy 107.95 85.09)
+		)
+		(stroke
+			(width 0)
+			(type default)
+		)
+	)
 	(wire
 		(pts
@@
 	(wire
 		(pts
-			(xy 107.95 78.74) (xy 107.95 85.09)
+			(xy 107.95 74.295) (xy 107.95 77.47)
 		)
 		(stroke
@@
 	(global_label "Input"
 		(shape input)
-		(at 107.95 78.74 90)
+		(at 107.95 74.295 90)
 		(fields_autoplaced yes)
 		(effects
@@
 		)
 		(property "Intersheetrefs" "${INTERSHEET_REFS}"
-			(at 107.95 70.9773 90)
+			(at 107.95 66.5323 90)
 			(hide yes)
 			(show_name no)
@@
 		(in_pos_files yes)
 		(dnp no)
-		(fields_autoplaced yes)
 		(property "Reference" "#PWR05"
 			(at 124.46 106.68 0)
@@
 		)
 		(property "Value" "GND"
-			(at 124.46 105.41 0)
+			(at 123.317 105.41 0)
 			(show_name no)
 			(do_not_autoplace no)
@@
 		(in_pos_files yes)
 		(dnp no)
-		(fields_autoplaced yes)
 		(property "Reference" "#PWR02"
 			(at 127 106.68 0)
@@
 		)
 		(property "Value" "GND"
-			(at 127 105.41 0)
+			(at 128.524 105.41 0)
 			(show_name no)
 			(do_not_autoplace no)
@@
 					(unit 1)
 				)
+			)
+		)
+	)
+	(symbol
+		(lib_id "Device:C_Small")
+		(at 107.95 80.01 0)
+		(mirror y)
+		(unit 1)
+		(body_style 1)
+		(exclude_from_sim no)
+		(in_bom yes)
+		(on_board yes)
+		(in_pos_files yes)
+		(dnp no)
+		(property "Reference" "C5"
+			(at 105.41 78.7462 0)
+			(show_name no)
+			(do_not_autoplace no)
+			(effects
+				(font
+					(size 1.27 1.27)
+				)
+				(justify left)
+			)
+		)
+		(property "Value" "1uF"
+			(at 105.41 81.2862 0)
+			(show_name no)
+			(do_not_autoplace no)
+			(effects
+				(font
+					(size 1.27 1.27)
+				)
+				(justify left)
+			)
+		)
+		(property "Footprint" ""
+			(at 107.95 80.01 0)
+			(hide yes)
+			(show_name no)
+			(do_not_autoplace no)
+			(effects
+				(font
+					(size 1.27 1.27)
+				)
+			)
+		)
+		(property "Datasheet" ""
+			(at 107.95 80.01 0)
+			(hide yes)
+			(show_name no)
+			(do_not_autoplace no)
+			(effects
+				(font
+					(size 1.27 1.27)
+				)
+			)
+		)
+		(property "Description" "Unpolarized capacitor, small symbol"
+			(at 107.95 80.01 0)
+			(hide yes)
+			(show_name no)
+			(do_not_autoplace no)
+			(effects
+				(font
+					(size 1.27 1.27)
+				)
+			)
+		)
+		(pin "2"
+		)
+		(pin "1"
+		)
+		(instances
+			(project "schematic"
+				(path "/6ada202e-a762-4b40-840a-77a412eabf67"
+					(reference "C5")
+					(unit 1)
+				)
